File: pcb/ish.kicad_pcb (KiCad board)
At the start: 2 copper layers, 275.5 x 105.6 mm, 117 parts, among them SW1 SW_PUSH, SW10 SW_PUSH, SW11 SW_PUSH, SW12 SW_PUSH, SW13 SW_PUSH, SW14 SW_PUSH, SW15 SW_PUSH, SW16 SW_PUSH, SW17 SW_PUSH, SW18 SW_PUSH, SW19 SW_PUSH, SW2 SW_PUSH, SW20 SW_PUSH, SW21 SW_PUSH, SW22 SW_PUSH, SW23 SW_PUSH, SW24 SW_PUSH, SW25 SW_PUSH, SW26 SW_PUSH, SW27 SW_PUSH, SW28 SW_PUSH, SW29 SW_PUSH, SW3 SW_PUSH, SW30 SW_PUSH, SW31 SW_PUSH, SW32 SW_PUSH, SW33 SW_PUSH, SW34 SW_PUSH, SW35 SW_PUSH, SW36 SW_PUSH, SW37 SW_PUSH, SW38 SW_PUSH, SW39 SW_PUSH, SW4 SW_PUSH, SW40 SW_PUSH, SW41 SW_PUSH, SW42 SW_PUSH, SW5 SW_PUSH, SW6 SW_PUSH, SW7 SW_PUSH, SW8 SW_PUSH, SW9 SW_PUSH, U1 ProMicro, U2 ProMicro

Commit message: hopefully rev 0.1.0 with new battery hookup and minor placement tweaks elsewhere
Parts:
- removed the REF** at (132.3, 63.9)
- removed the REF** at (159.9, 63.6)
- added REF**: Battery Pads, ish:Battery Pads, F.Cu at (162.0, 38.9)
- added REF**: Battery Pads, ish:Battery Pads, F.Cu at (135.1, 38.9)
- moved REF** 9.43 mm to (162.0, 46.4)
- moved REF** 9.03 mm to (134.8, 46.1)
- moved D32 6.25 mm to (197.1, 44.4)
- moved D28 5.45 mm to (272.8, 49.2)
- moved D33 4.22 mm to (175.8, 46.3)
- moved D10 3.64 mm to (85.4, 53.0)
- moved D29 3.32 mm to (249.5, 49.0)
- moved D20 2.85 mm to (97.0, 79.3)
- moved D21 2.78 mm to (100.6, 79.3)
- moved D19 2.63 mm to (93.2, 79.2)
- moved D41 2.56 mm to (193.9, 83.1)
- moved D30 2.55 mm to (230.3, 44.5)
- moved D42 2.55 mm to (190.3, 83.1)
- moved D40 2.43 mm to (197.5, 83.0)
- moved D34 1.66 mm to (266.6, 71.4)
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Routing:
- net row0_r: track 169.8 -> 129.5 mm, vias 2 -> 0
- net Net-(D42-Pad2): track 57.8 -> 25.0 mm
- net R-B+: track 12.9 -> 40.2 mm, vias 1 -> 2
- net L-B+: track 16.1 -> 40.3 mm, vias 0 -> 2
- net RAW: track 42.3 -> 56.8 mm, vias 0 -> 2
- net GNDA: track 0.00 -> 7.63 mm
- net GND: track 0.00 -> 7.55 mm
- net row1: track 118.1 -> 111.0 mm
- net Net-(D32-Pad2): track 3.83 -> 10.6 mm
- net RAW_R: track 61.5 -> 54.9 mm, vias 0 -> 2
- net col2: track 135.3 -> 141.8 mm
- net col1: track 158.3 -> 164.6 mm
- net Net-(D28-Pad2): track 4.40 -> 10.7 mm
- net col0: track 180.0 -> 185.8 mm
- net row2_r: track 137.1 -> 131.3 mm
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- removed copper zone on B.Cu, net GND
- removed copper zone on B.Cu, net GNDA
Other:
- outline, holes or cut-outs redrawn
- board text removed: "B+"
- board text removed: "B-"
