File: pcb/ish.kicad_pcb (KiCad board)
At the start: 2 copper layers, 275.5 x 105.6 mm, 117 parts, among them SW1 SW_PUSH, SW10 SW_PUSH, SW11 SW_PUSH, SW12 SW_PUSH, SW13 SW_PUSH, SW14 SW_PUSH, SW15 SW_PUSH, SW16 SW_PUSH, SW17 SW_PUSH, SW18 SW_PUSH, SW19 SW_PUSH, SW2 SW_PUSH, SW20 SW_PUSH, SW21 SW_PUSH, SW22 SW_PUSH, SW23 SW_PUSH, SW24 SW_PUSH, SW25 SW_PUSH, SW26 SW_PUSH, SW27 SW_PUSH, SW28 SW_PUSH, SW29 SW_PUSH, SW3 SW_PUSH, SW30 SW_PUSH, SW31 SW_PUSH, SW32 SW_PUSH, SW33 SW_PUSH, SW34 SW_PUSH, SW35 SW_PUSH, SW36 SW_PUSH, SW37 SW_PUSH, SW38 SW_PUSH, SW39 SW_PUSH, SW4 SW_PUSH, SW40 SW_PUSH, SW41 SW_PUSH, SW42 SW_PUSH, SW5 SW_PUSH, SW6 SW_PUSH, SW7 SW_PUSH, SW8 SW_PUSH, SW9 SW_PUSH, U1 ProMicro, U2 ProMicro

Commit message: ish v2.0.0
- now supports both MX and Choc v1 switches which can be used at the same time
- MCU is chips-down again to match the industry
- new smaller power and reset switches that fit under the pcb without
  adding thickness
- battery is connected via a reenforced JST

- support for an electronics cover has been _removed_
- with the MCU chips down, it is unwise to store the battery under the
  MCU. recommendation is to run the wires from the JST under the MCU,
  down through the cut out to a battery elsewhere
Parts:
- removed BATSWITCH1, BATSWITCH2: 1825232-1_TEC, ish:1825232-1
- removed the REF** at (135.1, 42.9)
- removed the REF** at (162.0, 42.9)
- removed RSW1, RSW2: SW_PUSH, ish:ResetSW_1side
- removed the Ref** at (154.4, 82.8)
- removed the Ref** at (168.9, 74.3)
- removed the Ref** at (127.9, 74.3)
- removed the Ref** at (142.3, 82.8)
- added REF**: CONN2_S02B-XASS_295x496_JST, ish:CONN2_S02B-XASS_295x496_JST, F.Cu at (136.1, 75.0)
- added REF**: SW_PCM12SMTR, ish:SW_PCM12SMTR, B.Cu at (142.1, 66.9)
- added REF**: SW_PCM12SMTR, ish:SW_PCM12SMTR, B.Cu at (154.8, 66.9)
- added REF**: EVQ_P7_PAN, ish:EVQ_P7_PAN-M, B.Cu at (142.5, 76.5)
- added REF**: EVQ_P7_PAN, ish:EVQ_P7_PAN-M, B.Cu at (154.1, 76.5)
- added REF**: CONN2_S02B-XASS_295x496_JST, ish:CONN2_S02B-XASS_295x496_JST, F.Cu at (163.2, 75.0)
- SW1, SW10, SW11, SW12, SW13, SW14, SW15, SW16, SW17, SW18, SW19, SW2, SW20, SW22, SW23, SW24, SW25, SW26, SW27, SW28, SW29, SW3, SW30, SW31, SW32, SW33, SW34, SW35, SW36, SW37, SW38, SW39, SW4, SW40, SW41, SW5, SW6, SW7, SW8, SW9: footprint ish:ChocV1_V2_Hotswap -> ish:CherryMX_MidHeight_Choc_Hotswap
- SW21, SW42: footprint ish:ChocV1_V2_Hotswap_1.5u -> ish:CherryMX_MidHeight_Choc_Hotswap
- U1, U2: footprint ish:ProMicro_v3 -> ish:ProMicro_v3 Chips Down
- moved REF** 45.0 mm to (134.8, 33.2)
- moved REF** 44.7 mm to (162.1, 33.4)
- moved D20 25.4 mm to (115.8, 96.4)
- moved D21 25.2 mm to (119.0, 96.4)
- moved D40 22.2 mm to (219.6, 85.4), turned to 90 degrees
- moved D30 18.3 mm to (245.6, 54.6), turned to 90 degrees
- moved D39 18.3 mm to (188.7, 77.3), turned to 90 degrees
- moved D10 18.2 mm to (70.3, 42.8)
- moved D34 18.1 mm to (283.4, 78.5), turned to 90 degrees
- moved D4 18.0 mm to (70.3, 24.1)
- moved D31 18.0 mm to (226.8, 53.5), turned to 90 degrees
- moved D24 17.8 mm to (245.9, 35.9), turned to 90 degrees
- moved D37 17.7 mm to (226.7, 72.7), turned to 90 degrees
- moved D36 17.7 mm to (245.6, 74.5), turned to 90 degrees
- moved D25 17.7 mm to (226.7, 34.9), turned to 90 degrees
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Connections:
- U1 pad 2: (no net) -> data1-L
- U2 pad 2: (no net) -> data1-R
Routing:
- net row1: track 111.9 -> 226.9 mm
- net row0: track 108.7 -> 220.2 mm
- net row2: track 131.1 -> 223.3 mm, vias 2 -> 0
- net col5: track 129.5 -> 78.1 mm
- net row1_r: track 148.9 -> 199.6 mm
- net col4: track 151.6 -> 103.8 mm, vias 8 -> 7
- net col3: track 170.3 -> 127.1 mm, vias 8 -> 7
- net row3_r: track 63.1 -> 99.4 mm, vias 0 -> 2
- net reset: track 34.4 -> 70.1 mm, vias 1 -> 2
- net row3: track 58.4 -> 91.3 mm, vias 2 -> 0
- net Net-(D42-Pad2): track 25.0 -> 57.2 mm, vias 0 -> 2
- net reset_r: track 37.9 -> 64.1 mm
- net row2_r: track 132.7 -> 158.2 mm, vias 0 -> 2
- net R-B+: track 36.1 -> 11.3 mm, vias 2 -> 0
- net L-B+: track 34.1 -> 9.70 mm, vias 2 -> 0
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Other:
- outline, holes or cut-outs redrawn
- board text added: "The ish keyboard https://git.sr.ht/~sungo/ish Yet another Corne-ish keyboard MIT License"
- board text removed: "The ish keyboard https://git.sr.ht/~sungo/ish Yet another Corne-ish keyboard Based on the Corne v3 keyboard by foostan - https://github.com/foostan/crkbd - https://github.com/foostan/kbd MIT License"

Commit message: add a signal led
Parts:
- added REF**: 4960_ADA, ish:SK6812MINI-E, B.Cu at (128.3, 72.1)
- added REF**: 4960_ADA, ish:SK6812MINI-E, B.Cu at (168.4, 72.1)
Connections:
- U1 pad 1: (no net) -> DIN-L
- U2 pad 1: (no net) -> DIN-R
Routing:
- net DIN-L: track 0.00 -> 65.8 mm
- net DIN-R: track 0.00 -> 45.4 mm, vias 0 -> 2
- net VCC: track 0.00 -> 42.7 mm, vias 0 -> 2
- net VDD: track 0.00 -> 38.2 mm, vias 0 -> 2
- net GND: track 17.3 -> 3.49 mm, vias 0 -> 2
- net GNDA: track 9.82 -> 3.25 mm, vias 0 -> 2
- net reset: track 70.1 -> 72.1 mm
- net row2_r: track 158.2 -> 156.4 mm
- net row3_r: track 99.4 -> 97.6 mm
- net row2: track 223.3 -> 225.1 mm
- net row3: track 91.3 -> 93.0 mm
- net reset_r: track 64.1 -> 65.1 mm
- net DOUT-L: track 0.00 -> 0.63 mm

Commit message: put the cover screw holes back
required moving things around a little and doing some routing that I'm
not super thrilled with. (The signal led's fault, tbh.) I _think_ I got
the screw holes in the right place.
Parts:
- added Ref**: Val**, ish:M2_HOLE_v2, F.Cu at (127.9, 74.2)
- added Ref**: Val**, ish:M2_HOLE_v2, F.Cu at (142.3, 82.8)
- added Ref**: Val**, ish:M2_HOLE_v2, F.Cu at (154.5, 82.8)
- added Ref**: Val**, ish:M2_HOLE_v2, F.Cu at (169.0, 74.2)
- moved REF** 4.62 mm to (128.3, 67.4), turned to 90 degrees
- moved REF** 4.62 mm to (168.4, 67.4), turned to 90 degrees
- moved REF** 2.00 mm to (163.2, 73.0)
- moved REF** 2.00 mm to (136.1, 73.0)
- moved REF** 1.00 mm to (142.5, 75.5)
- moved REF** 1.00 mm to (154.1, 75.5)
Connections:
- REF** pad 1: reset_r -> (no net)
- REF** pad 1*: (no net) -> reset_r
Routing:
- net reset_r: track 65.1 -> 38.4 mm, vias 2 -> 0
- net row3_r: track 97.6 -> 121.6 mm
- net row2_r: track 156.4 -> 177.9 mm
- net DIN-L: track 65.8 -> 44.3 mm, vias 0 -> 2
- net DIN-R: track 45.4 -> 34.6 mm
- net VCC: track 42.7 -> 32.7 mm
- net reset: track 72.1 -> 64.2 mm
- net R-B+: track 11.3 -> 15.4 mm
- net L-B+: track 9.70 -> 7.69 mm
- net col0: track 181.0 -> 179.0 mm
- net col1: track 151.5 -> 149.6 mm
- net col3: track 127.1 -> 125.3 mm
- net col2: track 127.4 -> 125.7 mm
- net col4: track 103.8 -> 102.1 mm
- net col5_r: track 89.9 -> 91.2 mm
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